File: bldc_controller.sch (KiCad schematic (older format))
At the start: 155 parts, among them J1 Barrel_Jack, J2 Conn_01x07, Q1 IRF4905, Q10 Q_NMOS_SGD, Q11 Q_NMOS_SGD, Q2 2N3904, Q3 IRLB8721PBF, Q4 IRLB8721PBF, Q5 IRLB8721PBF, Q6 IRLB8721PBF, Q7 IRLB8721PBF, Q8 IRLB8721PBF, Q9 Q_PMOS_SDG, SW1 D6C40 F1 LFS, SW2 D6C40 F1 LFS, SW3 1301.9314, U1 uA7810, U10 IRS2004, U11 LM339, U12 MCP601-xP, U13 LM319, U2 LM7805_TO220, U3 74LVC2G08, U4 CD4044BE, U6 ATmega328P-PU, U7 LM35-D, U8 IRS2004, U9 IRS2004, Y1 9B-16.000MBBK-B

Commit message: Update Schematic
Parts:
- removed U4: CD4044BE, DIP254P762X508-16, symbol CD4044BE:CD4044BE
- added R? (x6): 100K, symbol Device:R_US
Connections:
- wire segments 321 -> 324
Other:
- moved on the sheet: TP2, TP5, TP8

Commit message: Basically Ready for Layout
Parts:
- removed C22: 0.1uF, symbol Device:C
- removed C35: 0.1uF, symbol Device:C_Small
- removed D10, D8, D9: Green, symbol Device:LED
- removed D14: Red, symbol Device:LED
- removed D15: 5V Zener, symbol Device:D_Zener
- removed FB2: Ferrite_Bead, symbol Device:Ferrite_Bead
- removed J2: Conn_01x07, symbol Connector_Generic:Conn_01x07
- removed R18: 100, symbol Device:R_US
- removed R42: 1K, symbol Device:R_US
- removed R43: 576K, symbol Device:R_US
- removed RV1: 100K, symbol Device:R_POT
- removed SW3: 1301.9314, symbol Switch:SW_Push
- removed TP16, TP17, TP18, TP20, TP22: TestPoint, symbol Connector:TestPoint
- removed U13: LM319, symbol Comparator:LM319
- removed U7: LM35-D, Package_SO:SOIC-8_3.9x4.9mm_P1.27mm, symbol Sensor_Temperature:LM35-D
- added D3, D4, D6: LTST-C171GKT, symbol Device:LED
- added D5: LTST-C171KRKT, symbol Device:LED
- added J1: Conn_01x06_Male, symbol Connector:Conn_01x06_Male
- added R49: 1, symbol Device:R_US
- added SW1: 1301.9314, symbol Switch:SW_Push
- added U5: CD4044BE, N16, symbol CD4044BE:CD4044BE
- C5: renamed from C7; Part Number (none) -> EKY-101ETD470MJC5S
- D1: renamed from D7; value Green -> LTST-C171GKT; Color (none) -> Green
- D2: renamed from D11; value Red -> LTST-C171KRKT; Color (none) -> Red
- D9: renamed from D18; value Blue -> LTST-C171TBKT; Color (none) -> Blue
- F1: Part Number (none) -> 0685T5000-01; Size (none) -> 1206
- FB1: value Ferrite_Bead -> BL01RN1A1D2B
- J2: renamed from J1; value Barrel_Jack -> Banana_Jack
- Q1: renamed from Q9; value Q_PMOS_SDG -> FDN340P
- Q2: renamed from Q10; value Q_NMOS_SGD -> DMN65D8L-7
- Q3: renamed from Q11; value Q_NMOS_SGD -> DMN65D8L-7
- gave numbers to parts that had none: 6
- renumbered C13 to C1, C11 to C10, C2 to C11, C16 to C12, C9 to C13, C12 to C14, C3 to C15, C50 to C16, C4 to C17, C19 to C18, C20 to C19, C15 to C2, C5 to C20, C6 to C21, C34 to C22, C25 to C24, C27 to C25, C33 to C26, C30 to C27, C24 to C28, C26 to C29, C21 to C3, C28 to C30, C29 to C33, C1 to C4, C10 to C6, C17 to C7, C18 to C8, C8 to C9, D5 to D10, D6 to D11, D2 to D12, D4 to D13, D16 to D14, D17 to D15, D18 to D16, D1 to D7, D3 to D8, Q7 to Q10, Q8 to Q11, Q2 to Q4, Q1 to Q5, Q3 to Q6, Q4 to Q7, Q5 to Q8, Q6 to Q9, R10 to R1, R13 to R10, R7 to R11, R9 to R12, R44 to R13, R5 to R14, R51 to R15, R39 to R16, R4 to R17, R1 to R18, R3 to R19, R14 to R2, R2 to R20, R28 to R21, R41 to R22, R40 to R23, R29 to R24, R30 to R25, R19 to R26, R22 to R27, R25 to R28, R31 to R29, R11 to R3, R32 to R30, R20 to R31, R21 to R33, R23 to R35, R24 to R37, R26 to R39, R46 to R4, R27 to R41, R33 to R43, R34 to R44, R35 to R45, R36 to R46, R37 to R47, R38 to R48, R12 to R5, R8 to R7, R17 to R8, R45 to R9, RV2 to RV1, SW1 to SW2, SW2 to SW3, TP23 to TP1, TP4 to TP10, TP7 to TP11, TP19 to TP12, TP11 to TP13, TP12 to TP14, TP13 to TP15, TP10 to TP16, TP3 to TP17, TP6 to TP18, TP9 to TP19, TP14 to TP2, TP21 to TP3, TP15 to TP4, TP24 to TP5, TP2 to TP6, TP5 to TP7, TP1 to TP9, U6 to U1, U3 to U2, U1 to U3, U2 to U4, U11 to U6, U12 to U7
Connections:
- net labels removed: I_TRIG
- wire segments 324 -> 292
- no-connect marks 11 -> 6
Other:
- note removed: "CURRENT CONTROL"
- note removed: "Current Protection"
- note removed: "LED Indicators"
- note removed: "TEMPERATURE"
- moved on the sheet: C16, C22, R15, R16, RV1, TP2, TP3, TP4, U6D

Commit message: Ready for Layout
Parts:
- removed R49: 1, symbol Device:R_US
- removed TP1: TestPoint, symbol Connector:TestPoint
- removed U2: 74LVC2G08, symbol 74xGxx:74LVC2G08
- added J3: Banana_Jack, TestPoint:TestPoint_THTPad_D4.0mm_Drill2.0mm, symbol Connector:Barrel_Jack
- added JP1: SolderJumper_2_Open, Jumper:Solder_Jumper_2_Pin_5A, symbol Jumper:SolderJumper_2_Open
- added U2: SN74LVC1G11DBVR, Package_TO_SOT_SMD:SOT-23-6_Handsoldering, symbol SN74LVC1G11DBVR:SN74LVC1G11DBVR
- C1, C12, C13, C14, C15, C16, C17, C18, C19, C2, C20, C21, C22, C23, C24, C25, C26, C27, C28, C29, C3, C30, C31, C32, C33, C7, C8: footprint (none) -> Capacitor_SMD:C_0805_2012Metric_Pad1.15x1.40mm_HandSolder
- C10, C11, C4, C5, C6, C9: footprint (none) -> Capacitor_THT:CP_Radial_D10.0mm_P5.00mm
- D1, D2, D3, D4, D5, D6, D9: footprint (none) -> LED_SMD:LED_0805_2012Metric_Pad1.15x1.40mm_HandSolder
- D12, D13, D8: footprint (none) -> Diode_THT:D_DO-35_SOD27_P7.62mm_Horizontal
- F1: footprint (none) -> Fuse:Fuse_1206_3216Metric_Pad1.42x1.75mm_HandSolder
- FB1: footprint (none) -> Ferrite_THT:Ferrite_Bead_TH
- J1: footprint (none) -> Connector_PinHeader_2.54mm:PinHeader_1x06_P2.54mm_Vertical
- J2: footprint (none) -> TestPoint:TestPoint_THTPad_D4.0mm_Drill2.0mm
- Q1, Q2, Q3: footprint (none) -> Package_TO_SOT_SMD:SOT-23
- R1, R10, R11, R12, R13, R14, R15, R16, R17, R18, R19, R2, R20, R22, R23, R26, R27, R28, R3, R31, R32, R33, R34, R35, R36, R37, R38, R39, R4, R40, R41, R42, R43, R44, R45, R46, R47, R48, R5, R6, R7, R8, R9, RV1: footprint (none) -> Resistor_SMD:R_0805_2012Metric_Pad1.15x1.40mm_HandSolder
- R21, R24, R25, R29, R30: footprint (none) -> Resistor_THT:Power_Resistor_TH
- SW1: footprint (none) -> Button_Switch_SMD:Tactile_Switch_SM
- SW2: value D6C40 F1 LFS -> D6C50 F1 LFS; footprint (none) -> Button_Switch_THT:Pushbutton_Switch_TH
- SW3: footprint (none) -> Button_Switch_THT:Pushbutton_Switch_TH
- TP10, TP11, TP12, TP13, TP14, TP15, TP16, TP17, TP18, TP19, TP2, TP3, TP4, TP5, TP6, TP7, TP8, TP9: footprint (none) -> TestPoint:TestPoint_THTPad_1.0x1.0mm_Drill0.5mm
- U10, U8, U9: footprint (none) -> Package_DIP:DIP-8-16_W7.62mm
- U3: footprint (none) -> Package_TO_SOT_THT:TO-220-3_Vertical
- U5: footprint N16 -> Package_DIP:DIP-16_W7.62mm
- U6: footprint (none) -> Package_DIP:DIP-14_W7.62mm
- Y1: footprint (none) -> Crystal:Crystal_16MHz_TH
Connections:
- wire segments 292 -> 291
Other:
- moved on the sheet: C12, C16, C2, D11, J1, J2, R12, R15, R7, SW3

Commit message: Ready to Route
Parts:
- removed C10, C5, C6, C9: 47uF, Capacitor_THT:CP_Radial_D10.0mm_P5.00mm, symbol Device:CP
- removed D7: 1N62xxCA, Diode_THT:D_DO-201AE_P15.24mm_Horizontal, symbol Diode:1N62xxCA
- removed Q1: FDN340P, Package_TO_SOT_SMD:SOT-23, symbol Device:Q_PMOS_SDG
- removed Q2, Q3: DMN65D8L-7, Package_TO_SOT_SMD:SOT-23, symbol Device:Q_NMOS_SGD
- removed Q4: 2N3904, Package_TO_SOT_THT:TO-92_Inline, symbol Transistor_BJT:2N3904
- removed TP17, TP18, TP19: TestPoint, TestPoint:TestPoint_THTPad_1.0x1.0mm_Drill0.5mm, symbol Connector:TestPoint
- added C34, C35, C36: 0.47uF, Capacitor_SMD:C_0805_2012Metric_Pad1.15x1.40mm_HandSolder, symbol Device:C
- added C5: 0.33uF, Capacitor_SMD:C_0805_2012Metric_Pad1.15x1.40mm_HandSolder, symbol Device:C
- added C6: 0.22uF, Capacitor_SMD:C_0805_2012Metric_Pad1.15x1.40mm_HandSolder, symbol Device:C
- added Q1: 2N7002E, Package_TO_SOT_SMD:SOT-23, symbol Transistor_FET:2N7002E
- added Q2, Q3: DMN65D8L-7, Package_TO_SOT_SMD:SOT-23, symbol Transistor_FET:DMN67D7L
- added Q4: MMBT3904, Package_TO_SOT_SMD:SOT-23, symbol Transistor_BJT:MMBT3904
- added R49, R50, R51: 1K, Resistor_SMD:R_0805_2012Metric_Pad1.15x1.40mm_HandSolder, symbol Device:R_US
- D10, D11: value 1N914 -> BAT54HT1G; footprint Diode_THT:D_DO-35_SOD27_P7.62mm_Horizontal -> Diode_SMD:D_SOD-323_HandSoldering
- D12: value 13V Zener -> SMF12A; footprint Diode_THT:D_DO-35_SOD27_P7.62mm_Horizontal -> Diode_SMD:D_SOD-123F
- D13: value 6V Zener -> SMF5.0A; footprint Diode_THT:D_DO-35_SOD27_P7.62mm_Horizontal -> Diode_SMD:D_SOD-123F
- D14, D15, D16: value 1N5818 -> 1N5819; footprint Diode_THT:D_DO-41_SOD81_P10.16mm_Horizontal -> Diode_SMD:D_SOD-123
- D8: value 11V Zener -> SMF10A; footprint Diode_THT:D_DO-35_SOD27_P7.62mm_Horizontal -> Diode_SMD:D_SOD-123F
- J2, J3: footprint TestPoint:TestPoint_THTPad_D4.0mm_Drill2.0mm -> Connector_BarrelJack:BarrelJack_CUI_PJ-063AH_Horizontal
- RV1: footprint Resistor_SMD:R_0805_2012Metric_Pad1.15x1.40mm_HandSolder -> Potentiometer_THT:Potentiometer_Bourns_3339P_Vertical_HandSoldering
- U10, U8, U9: footprint Package_DIP:DIP-8-16_W7.62mm -> Package_DIP:DIP-8_W7.62mm
Connections:
- net labels added: Vdrive
- net labels removed: I_SET, T_SENSE
- wire segments 291 -> 289
- no-connect marks 6 -> 8
Other:
- moved on the sheet: C21, C33, D12, D5, D9, JP1, Q5, R13, R17, R18, R19, R20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

Commit message: Done with First Pass of Layout
Changed lines of the file:
@@
 	5200 8150 5800 8150
 Wire Wire Line
-	5200 7350 5800 7350
+	5200 7550 5800 7550
 Wire Wire Line
 	5200 7450 5800 7450
 Wire Wire Line
-	5200 7550 5800 7550
+	5200 7350 5800 7350
 Wire Wire Line
 	5200 7650 5800 7650
@@
 Text Label 5350 9550 0    50   ~ 0
 BEMF_A
-Text Label 5350 7250 0    50   ~ 0
-BEMF_B
 Text Label 5350 9650 0    50   ~ 0
+BEMF_B
+Text Label 5350 7250 0    50   ~ 0
 BEMF_C
 Text Label 5350 8450 0    50   ~ 0
@@
 	5200 9550 5800 9550
 Wire Wire Line
-	5200 9650 5800 9650
+	5200 7250 5800 7250
 Wire Wire Line
 	5200 8450 5800 8450
@@
 Text Label 5350 7750 0    50   ~ 0
 MCU_A_EN
-Text Label 5350 7550 0    50   ~ 0
+Text Label 5350 7350 0    50   ~ 0
 MCU_B_SIG
 Text Label 5350 7450 0    50   ~ 0
 MCU_C_SIG
-Text Label 5350 7350 0    50   ~ 0
+Text Label 5350 7550 0    50   ~ 0
 MCU_A_SIG
 Text Label 5350 8150 0    50   ~ 0
@@
 NoConn ~ 5200 8350
 Wire Wire Line
-	5200 7250 5800 7250
+	5200 9650 5800 9650
 NoConn ~ 5200 9450
 Wire Wire Line

Commit message: Added some shapes
Parts:
- removed J2, J3: Banana_Jack, Connector_BarrelJack:BarrelJack_CUI_PJ-063AH_Horizontal, symbol Connector:Barrel_Jack
- added FB2: BL01RN1A1D2B, Ferrite_THT:Ferrite_Bead_TH, symbol Device:Ferrite_Bead
- added J2: Screw_Terminal_01x04, Connector:Terminal_Block_4Pin_TH, symbol Connector:Screw_Terminal_01x04
Connections:
- wire segments 289 -> 292
Other:
- note added: "POWER"
Changed lines of the file:
@@
 	1    0    0    -1
 $EndComp
-Wire Wire Line
-	1500 1100 1700 1100
-$Comp
-L power:GNDPWR #PWR09
-U 1 1 5DC45516
-P 1700 1100
-F 0 "#PWR09" H 1700 900 50  0001 C CNN
-F 1 "GNDPWR" H 1704 946 50  0000 C CNN
-F 2 "" H 1700 1050 50  0001 C CNN
-F 3 "" H 1700 1050 50  0001 C CNN
-	1    1700 1100
-	1    0    0    -1
-$EndComp
-Wire Wire Line
-	1500 900  1700 900
 $Comp
 L power:+BATT #PWR08
 U 1 1 5DC4550F
-P 1700 900
-F 0 "#PWR08" H 1700 750 50  0001 C CNN
-F 1 "+BATT" H 1715 1073 50  0000 C CNN
-F 2 "" H 1700 900 50  0001 C CNN
-F 3 "" H 1700 900 50  0001 C CNN
-	1    1700 900
+P 1700 1350
+F 0 "#PWR08" H 1700 1200 50  0001 C CNN
+F 1 "+BATT" H 1715 1523 50  0000 C CNN
+F 2 "" H 1700 1350 50  0001 C CNN
+F 3 "" H 1700 1350 50  0001 C CNN
+	1    1700 1350
 	1    0    0    -1
 $EndComp
@@
 F 3 "~" H 4100 1100 50  0001 C CNN
 	1    4100 1100
-	1    0    0    -1
-$EndComp
-$Comp
-L Connector:Barrel_Jack J2
-U 1 1 5DC45503
-P 1200 1000
-F 0 "J2" H 1257 1325 50  0000 C CNN
-F 1 "Banana_Jack" H 1257 1234 50  0000 C CNN
-F 2 "Connector_BarrelJack:BarrelJack_CUI_PJ-063AH_Horizontal" H 1250 960 50  0001 C CNN
-F 3 "~" H 1250 960 50  0001 C CNN
-	1    1200 1000
 	1    0    0    -1
 $EndComp
@@
 	11150 1750 11150 2000
 Wire Wire Line
-	7250 2700 8300 2700
+	7250 2700 7650 2700
 $Comp
 L CD4044BE:CD4044BE U5
@@
 	0    -1   -1   0
 $EndComp
-Wire Wire Line
-	1500 1800 1700 1800
 $Comp
 L power:GNDPWR #PWR0109
 U 1 1 5E79C61A
-P 1700 1800
-F 0 "#PWR0109" H 1700 1600 50  0001 C CNN
-F 1 "GNDPWR" H 1704 1646 50  0000 C CNN
-F 2 "" H 1700 1750 50  0001 C CNN
-F 3 "" H 1700 1750 50  0001 C CNN
-	1    1700 1800
-	1    0    0    -1
-$EndComp
-$Comp
-L Connector:Barrel_Jack J3
-U 1 1 5E79C62F
-P 1200 1700
-F 0 "J3" H 1257 2025 50  0000 C CNN
-F 1 "Banana_Jack" H 1257 1934 50  0000 C CNN
-F 2 "Connector_BarrelJack:BarrelJack_CUI_PJ-063AH_Horizontal" H 1250 1660 50  0001 C CNN
-F 3 "~" H 1250 1660 50  0001 C CNN
-	1    1200 1700
-	1    0    0    -1
-$EndComp
-Wire Wire Line
-	1500 1600 1700 1600
+P 1500 1750
+F 0 "#PWR0109" H 1500 1550 50  0001 C CNN
+F 1 "GNDPWR" H 1504 1596 50  0000 C CNN
+F 2 "" H 1500 1700 50  0001 C CNN
+F 3 "" H 1500 1700 50  0001 C CNN
+	1    1500 1750
+	1    0    0    -1
+$EndComp
 $Comp
 L Jumper:SolderJumper_2_Open JP1
@@
 L power:Vdrive #PWR0113
 U 1 1 5F201E09
-P 1700 1600
-F 0 "#PWR0113" H 1500 1450 50  0001 C CNN
-F 1 "Vdrive" H 1717 1773 50  0000 C CNN
-F 2 "" H 1700 1600 50  0001 C CNN
-F 3 "" H 1700 1600 50  0001 C CNN
-	1    1700 1600
+P 1950 1450
+F 0 "#PWR0113" H 1750 1300 50  0001 C CNN
+F 1 "Vdrive" H 1967 1623 50  0000 C CNN
+F 2 "" H 1950 1450 50  0001 C CNN
+F 3 "" H 1950 1450 50  0001 C CNN
+	1    1950 1450
 	1    0    0    -1
 $EndComp
@@
 Connection ~ 11800 4750
 Connection ~ 11600 4750
+$Comp
+L Device:Ferrite_Bead FB2
+U 1 1 5DD92F7E
+P 7800 2700
+F 0 "FB2" V 7600 2700 50  0000 C CNN
+F 1 "BL01RN1A1D2B" V 8000 2700 50  0000 C CNN
+F 2 "Ferrite_THT:Ferrite_Bead_TH" V 7730 2700 50  0001 C CNN
+F 3 "~" H 7800 2700 50  0001 C CNN
+	1    7800 2700
+	0    1    1    0
+$EndComp
+Wire Wire Line
+	7950 2700 8300 2700
+$Comp
+L Connector:Screw_Terminal_01x04 J2
+U 1 1 5DDB786E
+P 950 1450
+F 0 "J2" H 950 1700 50  0000 C CNN
+F 1 "Screw_Terminal_01x04" H 900 1150 50  0000 C CNN
+F 2 "Connector:Terminal_Block_4Pin_TH" H 950 1450 50  0001 C CNN
+F 3 "~" H 950 1450 50  0001 C CNN
+	1    950  1450
+	-1   0    0    -1
+$EndComp
+Wire Wire Line
+	1150 1350 1700 1350
+Wire Wire Line
+	1150 1550 1500 1550
+Wire Wire Line
+	1500 1550 1500 1650
+Text Notes 1200 1000 0    50   ~ 10
+POWER
+Wire Wire Line
+	1150 1650 1500 1650
+Connection ~ 1500 1650
+Wire Wire Line
+	1500 1650 1500 1750
+Wire Wire Line
+	1150 1450 1950 1450
 $EndSCHEMATC

Commit message: Finished Ground Planes
Parts:
- removed FB2: BL01RN1A1D2B, Ferrite_THT:Ferrite_Bead_TH, symbol Device:Ferrite_Bead
- added R52, R53: 0, Resistor_SMD:R_0805_2012Metric_Pad1.15x1.40mm_HandSolder, symbol Device:R_US
Connections:
- wire segments 292 -> 296
Changed lines of the file:
@@
 Connection ~ 11800 4750
 Connection ~ 11600 4750
-$Comp
-L Device:Ferrite_Bead FB2
-U 1 1 5DD92F7E
-P 7800 2700
-F 0 "FB2" V 7600 2700 50  0000 C CNN
-F 1 "BL01RN1A1D2B" V 8000 2700 50  0000 C CNN
-F 2 "Ferrite_THT:Ferrite_Bead_TH" V 7730 2700 50  0001 C CNN
-F 3 "~" H 7800 2700 50  0001 C CNN
-	1    7800 2700
-	0    1    1    0
-$EndComp
 Wire Wire Line
 	7950 2700 8300 2700
@@
 Wire Wire Line
 	1150 1450 1950 1450
+$Comp
+L Device:R_US R52
+U 1 1 5E2BCD4A
+P 7800 2600
+F 0 "R52" V 7700 2450 50  0000 C CNN
+F 1 "0" V 7700 2750 50  0000 C CNN
+F 2 "Resistor_SMD:R_0805_2012Metric_Pad1.15x1.40mm_HandSolder" V 7840 2590 50  0001 C CNN
+F 3 "~" H 7800 2600 50  0001 C CNN
+	1    7800 2600
+	0    1    1    0
+$EndComp
+$Comp
+L Device:R_US R53
+U 1 1 5E2DB525
+P 7800 2800
+F 0 "R53" V 7900 2650 50  0000 C CNN
+F 1 "0" V 7900 2950 50  0000 C CNN
+F 2 "Resistor_SMD:R_0805_2012Metric_Pad1.15x1.40mm_HandSolder" V 7840 2790 50  0001 C CNN
+F 3 "~" H 7800 2800 50  0001 C CNN
+	1    7800 2800
+	0    1    1    0
+$EndComp
+Wire Wire Line
+	7650 2600 7650 2700
+Wire Wire Line
+	7650 2700 7650 2800
+Connection ~ 7650 2700
+Wire Wire Line
+	7950 2600 7950 2700
+Connection ~ 7950 2700
+Wire Wire Line
+	7950 2700 7950 2800
 $EndSCHEMATC

Commit message: Almost Done with Layout V2
Parts:
- added C10: 1uF, Capacitor_SMD:C_0805_2012Metric_Pad1.15x1.40mm_HandSolder, symbol Device:C
- added C37: 0.1uF, Capacitor_SMD:C_0805_2012Metric_Pad1.15x1.40mm_HandSolder, symbol Device:C
- added C9: 22uF, Capacitor_SMD:C_0805_2012Metric_Pad1.15x1.40mm_HandSolder, symbol Device:C
Connections:
- wire segments 296 -> 299
Other:
- note added: "Voltage Generation & Protection"
- note removed: "Voltage Generation\n& Protection"
- moved on the sheet: C11, C15, C17, C20, C4, F1, FB1, JP1
